File: Displaypanel/Displaypanel.kicad_sch (KiCad schematic)
At the start: 6 parts, among them J1 D_Connector, SW1 SW_Push_Dual, SW2 SW_Push_Dual

Commit message: Updated Readme
Other:
- title: (none) -> DisplayPanel
Changed lines of the file:
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@@
 	(generator_version "9.0")
 	(paper "A4")
+	(title_block
+		(title "DisplayPanel")
+		(date "2025-08-15")
+		(rev "0.9")
+	)
 	(no_connect
 		(at 59.69 64.77)
