File: Controller/Controller.kicad_sch (KiCad schematic)
At the start: 16 parts, among them J1 Probe, J2 Sonde, J3 Power, J4 D_Connector, J5 HayRain 3 Way, J8 SCT013, K1 FINDER-36.11, Q1 BC337, U4 TSR_1-2433

Commit message: Updated KiCad Controller
Other:
- title: (none) -> Controller RainControl
Changed lines of the file:
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@@
 	(generator_version "9.0")
 	(paper "A4")
+	(title_block
+		(title "Controller RainControl")
+		(date "2025-08-14")
+		(rev "0.9")
+	)
 	(junction
 		(at 74.93 43.18)

Commit message: Footprints updated, AREF to VCC
Updated Footprints from updatet Libraries and connected AREF to VCC,
Rerouted
Connections:
- net VCC: now also A1.AREF
- no-connect marks 15 -> 14
Changed lines of the file:
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@@
-	)
-	(no_connect
-		(at 132.08 78.74)
 	)
 	(no_connect
@@
 			(effects
 				(font
+					(size 1.27 1.27)
+				)
+				(justify right)
+				(hide yes)
+			)
+		)
+	)
+	(global_label "VCC"
+		(shape input)
+		(at 132.08 78.74 180)
+		(fields_autoplaced yes)
+		(effects
+			(font
+				(size 1.27 1.27)
+			)
+			(justify right)
+		)
+		(property "Intersheetrefs" "${INTERSHEET_REFS}"
+			(at 125.4662 78.74 0)
+			(effects
+				(font
